File: Hardware/STM8_Flasher.kicad_pcb (KiCad board)
At the start: 2 copper layers, 39 x 19.5 mm, 24 parts, among them J1 SWIM_PORT, J2 UART_PORT, J3 Power, J4 ISP, SW1 PROG_BUTTON, U1 STM8S003F3P, U2 AT24CS64-SSHM, U3 MIC5205-3.3

Commit message: initial commit
Parts:
- moved U2 0.71 mm to (114.5, 129.5)
Routing:
- net GND: track 51.8 -> 46.2 mm
- net I2C_SCL: track 9.41 -> 11.1 mm
- net SWIM_INT: track 21.3 -> 22.1 mm
- net I2C_SDA: track 5.71 -> 6.37 mm
- net +3V3: track 63.9 -> 63.4 mm
