File: Hardware/STM8_Flasher.sch (KiCad schematic (older format))
At the start: 19 parts, among them J1 SWIM_PORT, J2 UART_PORT, SW1 PROG_BUTTON, U1 STM8S003F3P, U2 AT24CS64-SSHM

Commit message: using PWM HW instead of SPI
Parts:
- removed R2: 22, symbol R
- added C5: 1uF, Capacitors_SMD:C_0805, symbol C
- added C6: 10uF, Capacitors_SMD:C_0805, symbol C
- added J3: Power, Pin_Headers:Pin_Header_Straight_1x02_Pitch2.54mm, symbol Conn_01x02
- added J4: ISP, Pin_Headers:Pin_Header_Straight_1x03_Pitch2.54mm, symbol Conn_01x03
- added U3: MIC5205-3.3, TO_SOT_Packages_SMD:SOT-23-5, symbol MIC5205-3.3
- C1: value C -> 0.1uF; footprint (none) -> Capacitors_SMD:C_0805
- C2: value C -> 1uF; footprint (none) -> Capacitors_SMD:C_0805
- C3: value C -> 10uF; footprint (none) -> Capacitors_SMD:C_0805
- C4: footprint (none) -> Capacitors_SMD:C_0805
- D1, D2: footprint (none) -> LEDs:LED_0805
- J1, J2: footprint (none) -> Pin_Headers:Pin_Header_Straight_1x03_Pitch2.54mm
- R1, R3, R4, R5, R6, R7, R8: footprint (none) -> Resistors_SMD:R_0805
- SW1: footprint (none) -> Buttons_Switches_THT:SW_PUSH_6mm
Connections:
- net labels added: SWIM_OUT, VCC
- net labels removed: SWIM_MISO, SWIM_MOSI, SWIM_SPI_CLK
- wire segments 69 -> 91

Commit message: initial commit
Parts:
- added R2: 22, Resistors_SMD:R_0805, symbol R
Changed lines of the file:
@@
 Text GLabel 7000 4050 2    60   Input ~ 0
 SWIM_OUT
+$Comp
+L R R2
+U 1 1 59D5E22B
+P 8450 5000
+F 0 "R2" V 8243 5000 50  0000 C CNN
+F 1 "22" V 8334 5000 50  0000 C CNN
+F 2 "Resistors_SMD:R_0805" V 8380 5000 50  0001 C CNN
+F 3 "" H 8450 5000 50  0001 C CNN
+	1    8450 5000
+	0    1    1    0
+$EndComp
 $EndSCHEMATC

Commit message: update
Parts:
- C1, C2, C3, C4, C5, C6: symbol C -> device:C
- D1, D2: symbol LED -> device:LED
- J1, J2, J4: symbol Conn_01x03 -> STM8_Flasher-rescue:Conn_01x03-RESCUE-STM8_Flasher
- J3: symbol Conn_01x02 -> STM8_Flasher-rescue:Conn_01x02-RESCUE-STM8_Flasher
- R1, R2, R3, R4, R5, R6, R7, R8: symbol R -> device:R
- SW1: symbol SW_Push -> STM8_Flasher-rescue:SW_Push-RESCUE-STM8_Flasher
- U1: symbol STM8S003F3P -> STM8_Flasher-rescue:STM8S003F3P-RESCUE-STM8_Flasher
- U2: footprint Housings_SOIC:SOIC-8_3.9x4.9mm_Pitch1.27mm -> Housings_SSOP:TSSOP-8_4.4x3mm_Pitch0.65mm; symbol AT24CS64-SSHM -> memory:AT24CS64-SSHM
- U3: symbol MIC5205-3.3 -> regul:MIC5205-3.3
Connections:
- wire segments 91 -> 106
Changed lines of the file:
@@
-EESchema Schematic File Version 3
-LIBS:power
-LIBS:device
-LIBS:transistors
-LIBS:conn
-LIBS:linear
-LIBS:regul
-LIBS:74xx
-LIBS:cmos4000
-LIBS:adc-dac
-LIBS:memory
-LIBS:xilinx
-LIBS:microcontrollers
-LIBS:dsp
-LIBS:microchip
-LIBS:analog_switches
-LIBS:motorola
-LIBS:texas
-LIBS:intel
-LIBS:audio
-LIBS:interface
-LIBS:digital-audio
-LIBS:philips
-LIBS:display
-LIBS:cypress
-LIBS:siliconi
-LIBS:opto
-LIBS:atmel
-LIBS:contrib
-LIBS:valves
-LIBS:stm8
-LIBS:switches
+EESchema Schematic File Version 4
 LIBS:STM8_Flasher-cache
 EELAYER 26 0
@@
 $EndDescr
 $Comp
-L STM8S003F3P U1
+L STM8_Flasher-rescue:STM8S003F3P-RESCUE-STM8_Flasher U1
 U 1 1 59C0F5D5
 P 5500 3650
@@
 $EndComp
 $Comp
-L C C1
+L device:C C1
 U 1 1 59C0F653
 P 3500 4450
@@
 $EndComp
 $Comp
-L C C2
+L device:C C2
 U 1 1 59C0F6D1
 P 3850 4450
@@
 $EndComp
 $Comp
-L C C3
+L device:C C3
 U 1 1 59C0F723
 P 3000 2150
@@
 $EndComp
 $Comp
-L GND #PWR01
+L power:GND #PWR01
 U 1 1 59C0F95C
 P 5500 4700
@@
 	5500 4700 5500 4550
 $Comp
-L R R1
+L device:R R1
 U 1 1 59C0FA26
 P 8450 5350
@@
 	8800 5350 8800 5650
 Wire Wire Line
-	8600 5350 9600 5350
+	8600 5350 8800 5350
 Wire Wire Line
 	8300 5000 8150 5000
@@
 SWIM_INT
 $Comp
-L Conn_01x03 J1
+L STM8_Flasher-rescue:Conn_01x03-RESCUE-STM8_Flasher J1
 U 1 1 59C1001A
 P 10100 5350
@@
 Connection ~ 8800 5350
 $Comp
-L GND #PWR02
+L power:GND #PWR02
 U 1 1 59C10296
 P 9750 5550
@@
 	9750 5550 9750 5450
 $Comp
-L GND #PWR06
+L power:GND #PWR06
 U 1 1 59C1043A
 P 3850 4700
@@
 	3500 4300 3500 3150
 Wire Wire Line
-	3500 3150 4200 3150
-$Comp
-L GND #PWR05
+	3500 3150 4050 3150
+$Comp
+L power:GND #PWR05
 U 1 1 59C107C3
 P 3500 4700
@@
 	3000 1850 3000 2000
 $Comp
-L GND #PWR04
+L power:GND #PWR04
 U 1 1 59C108BF
 P 3000 2450
@@
 $EndComp
 $Comp
-L +3.3V #PWR03
+L power:+3.3V #PWR03
 U 1 1 59C10A13
 P 3000 1850
@@
 	3000 2450 3000 2300
 $Comp
-L +3.3V #PWR09
+L power:+3.3V #PWR09
 U 1 1 59C10D1C
 P 5500 2750
@@
 	5500 2750 5500 2850
 $Comp
-L Conn_01x03 J2
+L STM8_Flasher-rescue:Conn_01x03-RESCUE-STM8_Flasher J2
 U 1 1 59C10E6F
 P 10100 6000
@@
 	10300 6100 10500 6100
 $Comp
-L GND #PWR015
+L power:GND #PWR015
 U 1 1 59C11386
 P 10350 6250
@@
 	4100 3850 4200 3850
 $Comp
-L AT24CS64-SSHM U2
+L memory:AT24CS64-SSHM U2
 U 1 1 59C119A2
 P 9250 1900
 F 0 "U2" H 10100 1550 50  0000 C CNN
 F 1 "AT24CS64-SSHM" H 10050 1650 50  0000 C CNN
-F 2 "Housings_SOIC:SOIC-8_3.9x4.9mm_Pitch1.27mm" H 9250 1900 50  0001 C CIN
+F 2 "Housings_SSOP:TSSOP-8_4.4x3mm_Pitch0.65mm" H 9250 1900 50  0001 C CIN
 F 3 "" H 9250 1900 50  0001 C CNN
 	1    9250 1900
@@
 I2C_SDA
 Wire Wire Line
-	9650 1800 10000 1800
-Wire Wire Line
-	9650 1950 10000 1950
-$Comp
-L R R7
+	9650 1800 9900 1800
+Wire Wire Line
+	9650 1950 9700 1950
+$Comp
+L device:R R7
 U 1 1 59C11E85
 P 9900 1600
@@
 $EndComp
 $Comp
-L R R6
+L device:R R6
 U 1 1 59C11FBE
 P 9700 1350
@@
 $EndComp
 $Comp
-L +3.3V #PWR011
+L power:+3.3V #PWR011
 U 1 1 59C120BF
 P 9250 1450
@@
 	9250 1450 9250 1550
 $Comp
-L GND #PWR012
+L power:GND #PWR012
 U 1 1 59C122DA
 P 9250 2400
@@
 $EndComp
 Wire Wire Line
-	9250 2300 9250 2400
+	9250 2300 9250 2350
 Wire Wire Line
 	9900 1750 9900 1800
@@
 Connection ~ 9700 1950
 Wire Wire Line
-	9900 1100 9900 1450
+	9900 1100 9900 1150
 Wire Wire Line
 	9900 1150 9700 1150
@@
 	9700 1150 9700 1200
 $Comp
-L +3.3V #PWR014
+L power:+3.3V #PWR014
 U 1 1 59C1251C
 P 9900 1100
@@
 	8750 2100 8850 2100
 Wire Wire Line
-	8750 1750 8750 2350
+	8750 1750 8750 1850
 Wire Wire Line
 	8750 2350 9250 2350
@@
 	6800 3550 7000 3550
 $Comp
-L LED D2
+L device:LED D2
 U 1 1 59C12CAD
 P 10000 3900
@@
 $EndComp
 $Comp
-L LED D1
+L device:LED D1
 U 1 1 59C12F50
 P 9600 3900
@@
 $EndComp
 $Comp
-L R R8
+L device:R R8
 U 1 1 59C1305C
 P 10000 4300
@@
 $EndComp
 $Comp
-L R R5
+L device:R R5
 U 1 1 59C1314F
 P 9600 4300
@@
 	10000 3650 10000 3750
 Wire Wire Line
-	9600 3650 10000 3650
+	9600 3650 9800 3650
 Wire Wire Line
 	9600 3650 9600 3750
 $Comp
-L +3.3V #PWR013
+L power:+3.3V #PWR013
 U 1 1 59C13885
 P 9800 3550
@@
 	6800 3250 7000 3250
 $Comp
-L SW_Push SW1
+L STM8_Flasher-rescue:SW_Push-RESCUE-STM8_Flasher SW1
 U 1 1 59C14A74
 P 6250 1500
@@
 $EndComp
 $Comp
-L GND #PWR010
+L power:GND #PWR010
 U 1 1 59C14E89
 P 6550 1900
@@
 PROG_SWITCH
 $Comp
-L C C4
+L device:C C4
 U 1 1 59C1512B
 P 5400 1700
@@
 $EndComp
 $Comp
-L R R4
+L device:R R4
 U 1 1 59C1532B
 P 5750 1500
@@
 	5900 1500 6050 1500
 Wire Wire Line
-	5150 1500 5600 1500
-Wire Wire Line
-	5400 1350 5400 1550
+	5150 1500 5400 1500
+Wire Wire Line
+	5400 1350 5400 1500
 Connection ~ 5400 1500
 $Comp
-L GND #PWR08
+L power:GND #PWR08
 U 1 1 59C1562F
 P 5400 1950
@@
 	5400 1850 5400 1950
 $Comp
-L R R3
+L device:R R3
 U 1 1 59C15857
 P 5400 1200
@@
 $EndComp
 $Comp
-L +3.3V #PWR07
+L power:+3.3V #PWR07
 U 1 1 59C159E6
 P 5400 1000
@@
 PROG_SWITCH
 $Comp
-L MIC5205-3.3 U3
+L regul:MIC5205-3.3 U3
 U 1 1 59C527A2
 P 2000 3150
@@
 $EndComp
 Wire Wire Line
-	1300 3050 1700 3050
+	1300 3050 1500 3050
 Wire Wire Line
 	1500 3050 1500 3150
@@
 	1500 3150 1700 3150
 $Comp
-L VCC #PWR016
+L power:VCC #PWR016
 U 1 1 59C52BA0
 P 1300 2950
@@
 $EndComp
 Wire Wire Line
-	1300 2950 1300 3150
+	1300 2950 1300 3050
 Connection ~ 1500 3050
 $Comp
-L GND #PWR017
+L power:GND #PWR017
 U 1 1 59C52EC4
 P 2000 3550
@@
 	2000 3550 2000 3450
 $Comp
-L +3.3V #PWR018
+L power:+3.3V #PWR018
 U 1 1 59C53156
 P 2450 3000
@@
 	2300 3050 2450 3050
 Wire Wire Line
-	2450 3000 2450 3150
-$Comp
-L C C5
+	2450 3000 2450 3050
+$Comp
+L device:C C5
 U 1 1 59C533C2
 P 1300 3300
@@
 $EndComp
 $Comp
-L C C6
+L device:C C6
 U 1 1 59C53573
 P 2450 3300
@@
 $EndComp
 $Comp
-L GND #PWR019
+L power:GND #PWR019
 U 1 1 59C535D1
 P 1300 3550
@@
 $EndComp
 $Comp
-L GND #PWR020
+L power:GND #PWR020
 U 1 1 59C536A8
 P 2450 3550
@@
 Connection ~ 1300 3050
 $Comp
-L Conn_01x02 J3
+L STM8_Flasher-rescue:Conn_01x02-RESCUE-STM8_Flasher J3
 U 1 1 59C53E9C
 P 1300 2000
@@
 $EndComp
 $Comp
-L VCC #PWR021
+L power:VCC #PWR021
 U 1 1 59C5404D
 P 1700 1700
@@
 $EndComp
 $Comp
-L GND #PWR022
+L power:GND #PWR022
 U 1 1 59C540F9
 P 1700 2150
@@
 	9450 5450 9450 5250
 $Comp
-L Conn_01x03 J4
+L STM8_Flasher-rescue:Conn_01x03-RESCUE-STM8_Flasher J4
 U 1 1 59CB813E
 P 3700 2800
@@
 	4050 2800 3900 2800
 $Comp
-L GND #PWR023
+L power:GND #PWR023
 U 1 1 59CB84AF
 P 4250 2750
@@
 SWIM_OUT
 $Comp
-L R R2
+L device:R R2
 U 1 1 59D5E22B
 P 8450 5000
@@
 	0    1    1    0
 $EndComp
+Wire Wire Line
+	8800 5350 9600 5350
+Wire Wire Line
+	9900 1800 10000 1800
+Wire Wire Line
+	9700 1950 10000 1950
+Wire Wire Line
+	9900 1150 9900 1450
+Wire Wire Line
+	9250 2350 9250 2400
+Wire Wire Line
+	8750 2100 8750 2350
+Wire Wire Line
+	8750 1950 8750 2100
+Wire Wire Line
+	8750 1850 8750 1950
+Wire Wire Line
+	9800 3650 10000 3650
+Wire Wire Line
+	5400 1500 5600 1500
+Wire Wire Line
+	5400 1500 5400 1550
+Wire Wire Line
+	1500 3050 1700 3050
+Wire Wire Line
+	2450 3050 2450 3150
+Wire Wire Line
+	1300 3050 1300 3150
+Wire Wire Line
+	4050 3150 4200 3150
 $EndSCHEMATC

Commit message: schematic update
Parts:
- removed C1, C4: 0.1uF, Capacitors_SMD:C_0805, symbol device:C
- removed C2, C5: 1uF, Capacitors_SMD:C_0805, symbol device:C
- removed C3, C6: 10uF, Capacitors_SMD:C_0805, symbol device:C
- removed D1, D2: LED, LEDs:LED_0805, symbol device:LED
- removed J1: SWIM_PORT, Pin_Headers:Pin_Header_Straight_1x03_Pitch2.54mm, symbol STM8_Flasher-rescue:Conn_01x03-RESCUE-STM8_Flasher
- removed J2: UART_PORT, Pin_Headers:Pin_Header_Straight_1x03_Pitch2.54mm, symbol STM8_Flasher-rescue:Conn_01x03-RESCUE-STM8_Flasher
- removed J3: Power, Pin_Headers:Pin_Header_Straight_1x02_Pitch2.54mm, symbol STM8_Flasher-rescue:Conn_01x02-RESCUE-STM8_Flasher
- removed J4: ISP, Pin_Headers:Pin_Header_Straight_1x03_Pitch2.54mm, symbol STM8_Flasher-rescue:Conn_01x03-RESCUE-STM8_Flasher
- removed R1: 680, Resistors_SMD:R_0805, symbol device:R
- removed R2: 22, Resistors_SMD:R_0805, symbol device:R
- removed R3: 10k, Resistors_SMD:R_0805, symbol device:R
- removed R4: 1k, Resistors_SMD:R_0805, symbol device:R
- removed R5, R8: 330, Resistors_SMD:R_0805, symbol device:R
- removed R6, R7: 4.7k, Resistors_SMD:R_0805, symbol device:R
- removed SW1: PROG_BUTTON, Buttons_Switches_THT:SW_PUSH_6mm, symbol STM8_Flasher-rescue:SW_Push-RESCUE-STM8_Flasher
- removed U1: STM8S003F3P, Housings_SSOP:TSSOP-20_4.4x6.5mm_Pitch0.65mm, symbol STM8_Flasher-rescue:STM8S003F3P-RESCUE-STM8_Flasher
- removed U2: AT24CS64-SSHM, Housings_SSOP:TSSOP-8_4.4x3mm_Pitch0.65mm, symbol memory:AT24CS64-SSHM
- removed U3: MIC5205-3.3, TO_SOT_Packages_SMD:SOT-23-5, symbol regul:MIC5205-3.3
- added C1, C2, C3, C5: 1u, Capacitor_SMD:C_0805_2012Metric, symbol Device:C
- added C4: 10u, Capacitor_SMD:C_0805_2012Metric, symbol Device:C
- added C6: 0.1u, Capacitor_SMD:C_0805_2012Metric, symbol Device:C
- added D1, D2: LED, Capacitor_SMD:C_0805_2012Metric, symbol Device:LED
- added IC1: STM8S003F3P, Package_SO:TSSOP-20_4.4x6.5mm_P0.65mm, symbol stm8:STM8S003F3P
- added J1: SWIM_Port, Connector_PinHeader_2.54mm:PinHeader_1x03_P2.54mm_Vertical, symbol Connector_Generic:Conn_01x03
- added J2: ISP_Port, Connector_PinHeader_2.54mm:PinHeader_1x03_P2.54mm_Vertical, symbol Connector_Generic:Conn_01x03
- added J3: Power, Connector_PinHeader_2.54mm:PinHeader_1x02_P2.54mm_Vertical, symbol Connector_Generic:Conn_01x02
- added J4: UART_Port, Connector_PinHeader_2.54mm:PinHeader_1x03_P2.54mm_Vertical, symbol Connector_Generic:Conn_01x03
- added R1: 10k, Resistor_SMD:R_0805_2012Metric, symbol Device:R
- added R2, R4, R9: 1k, Resistor_SMD:R_0805_2012Metric, symbol Device:R
- added R3: 3.3k, Resistor_SMD:R_0805_2012Metric, symbol Device:R
- added R5, R6: 100, Resistor_SMD:R_0805_2012Metric, symbol Device:R
- added R7, R8: 4.7k, Resistor_SMD:R_0805_2012Metric, symbol Device:R
- added SW1: SW_Push, Button_Switch_THT:SW_PUSH_6mm, symbol Switch:SW_Push
- added U1: MIC5205-3.3YM5, Package_TO_SOT_SMD:SOT-23-5, symbol Regulator_Linear:MIC5205-3.3YM5
- added U2: 24LC256, Package_SO:TSSOP-8_4.4x3mm_P0.65mm, symbol Memory_EEPROM:24LC256
Connections:
- net labels removed: SWIM_INT
- wire segments 106 -> 98
